File: spice/doa4/kicad/doa4.kicad_pcb (KiCad board)
At the start: 2 copper layers, 34 parts, among them J1 CONN_01X06, Q1 BC557, Q10 BC547, Q11 BD139, Q12 BD140, Q2 BC557, Q3 BC547, Q4 BC547, Q5 BC557, Q6 BC547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

Commit message: location  q8q5 cont
Parts:
- moved RPCS1 30.9 mm to (66.2, 78.2)
- moved Q5 29.8 mm to (72.6, 85.0)
- moved Q8 29.6 mm to (72.4, 80.5)
- moved RE1 8.89 mm to (74.1, 98.9), turned to 90 degrees
- moved RCP1 8.45 mm to (67.5, 91.0)
- moved D5 4.98 mm to (71.2, 75.2), turned to 270 degrees
Routing:
- net /V+: track 41.0 -> 25.9 mm
- net Net-(Q10-Pad1): track 0.29 -> 12.6 mm
- net /Out: track 16.0 -> 25.7 mm
- net Net-(D6-Pad2): track 3.03 -> 12.1 mm
- net Net-(D5-Pad2): track 10.6 -> 19.2 mm
- net Net-(Q10-Pad3): track 0.00 -> 7.75 mm
- net /ODiff: track 9.53 -> 15.4 mm
- net Net-(Q4-Pad3): track 22.2 -> 27.9 mm
- net Net-(Cp1-Pad2): track 2.52 -> 6.88 mm
- net /V-: track 101.7 -> 105.0 mm
