File: spice/doa4/kicad/doa4.kicad_pcb (KiCad board)
At the start: 2 copper layers, 34 parts, among them J1 CONN_01X06, Q1 BC557, Q10 BC547, Q11 BD139, Q12 BD140, Q2 BC557, Q3 BC547, Q4 BC547, Q5 BC557, Q6 BC547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

Commit message: v1 complete
Parts:
- moved D3 31.4 mm to (74.1, 81.9)
- moved D4 27.8 mm to (67.9, 74.7)
- moved RCS1 26.7 mm to (74.4, 87.7), turned to 180 degrees
- moved D8 13.4 mm to (77.7, 89.9), turned to 180 degrees
- moved RE2 7.06 mm to (82.3, 73.4), turned to 270 degrees
- moved Q11 6.67 mm to (77.7, 79.0), turned to 90 degrees
- moved D7 6.13 mm to (82.0, 89.4), turned to 270 degrees
- moved Q12 5.46 mm to (77.2, 93.2), turned to 270 degrees
- moved D6 4.79 mm to (72.9, 91.7)
- moved RE3 3.68 mm to (80.8, 98.6), turned to 90 degrees
- moved D5 2.75 mm to (73.7, 73.9), turned to 0 degrees
- moved C5 0.59 mm to (82.0, 83.6)
- moved C4 0.55 mm to (82.0, 78.3)
Routing:
- net /Emiter: track 3.80 -> 47.0 mm
- net Net-(D5-Pad1): track 0.00 -> 20.2 mm
- net Net-(D5-Pad2): track 19.2 -> 35.2 mm
- net Net-(Q8-Pad3): track 0.00 -> 12.1 mm
- net /Out: track 25.7 -> 35.0 mm
- net /V+: track 25.9 -> 34.1 mm
- net /VrefCS: track 11.8 -> 19.2 mm
- net Net-(D3-Pad1): track 2.08 -> 8.72 mm
- net /V-: track 105.0 -> 109.2 mm
- net Net-(D6-Pad2): track 12.1 -> 9.61 mm
- net /ODiff: track 15.4 -> 17.9 mm
- net Net-(Q5-Pad3): track 4.58 -> 2.84 mm
- net Net-(Q12-Pad1): track 4.39 -> 3.66 mm
- net GND: track 5.85 -> 5.22 mm

Commit message: re-locating v1
Parts:
- moved RCS1 4.35 mm to (75.4, 83.4)
- moved D4 3.75 mm to (71.5, 73.7)
- moved D3 3.43 mm to (74.0, 78.5)
- moved RPCS1 2.17 mm to (67.1, 76.2), turned to 180 degrees
- moved Q8 1.96 mm to (72.5, 78.6)
- moved Q5 1.58 mm to (72.5, 83.4)
- moved RE1 1.32 mm to (74.9, 97.9)
- moved D6 1.08 mm to (73.7, 90.9)
- moved RE3 0.76 mm to (80.0, 98.6)
- moved RE2 0.28 mm to (82.0, 73.5)
- moved Q7 0.13 mm to (63.8, 84.1)
Routing:
- net /V-: track 109.2 -> 103.0 mm
- net Net-(D3-Pad1): track 8.72 -> 3.59 mm
- net Net-(Q11-Pad1): track 5.14 -> 9.62 mm
- net /V+: track 34.1 -> 38.1 mm
- net /VrefCS: track 19.2 -> 15.6 mm
- net Net-(D5-Pad1): track 20.2 -> 16.8 mm
- net /In-: track 11.6 -> 9.45 mm
- net Net-(D5-Pad2): track 35.2 -> 33.2 mm
- net /ODiff: track 17.9 -> 16.3 mm
- net /Out: track 35.0 -> 33.5 mm
- net Net-(Q5-Pad3): track 2.84 -> 1.56 mm
- net Net-(Q10-Pad3): track 7.75 -> 9.01 mm
- net Net-(Q12-Pad1): track 3.66 -> 2.90 mm
- net /Emiter: track 47.0 -> 47.6 mm

Commit message: re-locating v1 cont
Parts:
- moved RCP1 4.11 mm to (67.5, 86.9)
- moved RSZ3 2.07 mm to (69.8, 93.2)
- moved Q10 1.76 mm to (68.3, 100.2)
- moved D4 1.40 mm to (70.1, 73.7)
Routing:
- net /V+: track 38.1 -> 28.8 mm
- net Net-(Cp1-Pad2): track 6.88 -> 2.48 mm
- net /ODiff: track 16.3 -> 18.6 mm
- net Net-(Q10-Pad1): track 12.5 -> 14.3 mm
- net Net-(Q10-Pad3): track 9.01 -> 7.34 mm
- net Net-(D3-Pad1): track 3.59 -> 4.99 mm
- net Net-(D6-Pad2): track 9.66 -> 8.51 mm
- net Net-(Q8-Pad3): track 12.5 -> 11.4 mm

Commit message: re-locating v1 cont 2
Parts:
- moved D2 2.08 mm to (57.5, 88.4), turned to 270 degrees
- moved D1 2.04 mm to (57.3, 84.1)
Routing:
- net /In-: track 9.45 -> 13.3 mm
- net /ODiff: track 18.6 -> 17.4 mm
- net /In+: track 7.64 -> 8.76 mm
- net /Emiter: track 47.4 -> 48.4 mm

Commit message: re-locating v1 cont 2
Parts:
- moved RCS1 0.08 mm to (75.4, 83.4)
Changed lines of the file:
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@@
   (general
     (links 61)
-    (no_connects 1)
-    (area 52.478438 70.995038 84.4886 100.859001)
+    (no_connects 0)
+    (area 52.605438 70.995038 84.4886 100.859001)
     (thickness 1.6)
     (drawings 0)
@@
       (hpglpenoverlay 2)
       (psnegative false)
-      (psa4output true)
+      (psa4output false)
       (plotreference true)
       (plotvalue true)
@@
       (padsonsilk false)
       (subtractmaskfromsilk false)
-      (outputformat 2)
-      (mirror true)
-      (drillshape 1)
+      (outputformat 1)
+      (mirror false)
+      (drillshape 0)
       (scaleselection 1)
       (outputdirectory ./))
@@
   )
   (module Doa4FPLibrary:R_Axial_DIN0207_L6.3mm_D2.5mm_P2.54mm_Vertical_Doa4 (layer F.Cu)
-    (at 75.438 83.439 180)
+    (at 75.3618 83.439 180)
     (descr "Resistor, Axial_DIN0207 series, Axial, Vertical, pin pitch=2.54mm, 0.25W = 1/4W, length*diameter=6.3*2.5mm^2, http://cdn-reichelt.de/documents/datenblatt/B400/1_4W%23YAG.pdf")
     (tags "Resistor Axial_DIN0207 series Axial Vertical pin pitch 2.54mm 0.25W = 1/4W length 6.3mm diameter 2.5mm")
@@
     )
   )
+  (segment (start 80.01 79.093002) (end 76.214001 82.889001) (width 0.25) (layer B.Cu) (net 1))
+  (segment (start 75.911799 82.889001) (end 75.3618 83.439) (width 0.25) (layer B.Cu) (net 1))
+  (segment (start 76.214001 82.889001) (end 75.911799 82.889001) (width 0.25) (layer B.Cu) (net 1))
   (segment (start 70.104 73.66) (end 65.405 73.66) (width 0.25) (layer B.Cu) (net 1) (status 30))
   (segment (start 65.405 73.66) (end 65.151 73.406) (width 0.25) (layer B.Cu) (net 1) (status 30))
@@
   (segment (start 74.470001 73.038999) (end 71.525001 73.038999) (width 0.25) (layer B.Cu) (net 1))
   (segment (start 71.525001 73.038999) (end 70.904 73.66) (width 0.25) (layer B.Cu) (net 1))
-  (segment (start 75.438 83.439) (end 75.987999 82.889001) (width 0.25) (layer B.Cu) (net 1) (status 10))
   (segment (start 80.01 79.093002) (end 80.01 76.962) (width 0.25) (layer B.Cu) (net 1) (status 20))
-  (segment (start 75.987999 82.889001) (end 76.214001 82.889001) (width 0.25) (layer B.Cu) (net 1))
-  (segment (start 76.214001 82.889001) (end 80.01 79.093002) (width 0.25) (layer B.Cu) (net 1))
   (segment (start 80.01 76.962) (end 78.232 76.962) (width 0.25) (layer B.Cu) (net 1) (status 30))
   (segment (start 78.232 76.962) (end 77.724 76.454) (width 0.25) (layer B.Cu) (net 1) (status 30))
@@
   (segment (start 68.212999 80.391) (end 67.056 79.234001) (width 0.25) (layer B.Cu) (net 9))
   (segment (start 67.056 79.234001) (end 67.056 76.2) (width 0.25) (layer B.Cu) (net 9) (status 20))
-  (segment (start 73.279 83.439) (end 71.755 83.439) (width 0.25) (layer B.Cu) (net 10) (status 30))
-  (segment (start 71.755 83.439) (end 71.7296 83.4136) (width 0.25) (layer B.Cu) (net 10) (status 30))
+  (segment (start 73.2028 83.439) (end 71.755 83.439) (width 0.25) (layer B.Cu) (net 10))
+  (segment (start 71.755 83.439) (end 71.7296 83.4136) (width 0.25) (layer B.Cu) (net 10))
   (segment (start 63.754 83.312) (end 63.754 88.646) (width 0.25) (layer B.Cu) (net 11))
   (segment (start 63.754 88.646) (end 63.7286 88.6714) (width 0.25) (layer B.Cu) (net 11))

Commit message: RE nueva ubicacion
Parts:
- moved RE3 1.91 mm to (81.9, 98.4)
Routing:
- net Net-(Q12-Pad1): track 2.90 -> 5.11 mm
- net /Out: track 33.5 -> 35.3 mm
- net /Emiter: track 48.4 -> 47.6 mm
